File: pcb/plugnslay/clamp_couple.kicad_sch (KiCad schematic)
At the start: 11 parts, among them U2 ADA4622-2xCP

Commit message: complete first prototype
Parts:
- removed C6: 2.2u, symbol Device:C
- added C10: 2.2u, Capacitor_SMD:C_1206_3216Metric_Pad1.33x1.80mm_HandSolder, symbol Device:C
- D3, D4, D5, D6, D7, D8: footprint (none) -> Diode_SMD:D_SOD-123; Link (none) -> https://www.mouser.com/ProductDetail/Vishay/1N4448W-HE3_A-0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; Part Number (none) -> 1N4448W-HE3_A-08
- R14, R15: footprint (none) -> Resistor_SMD:R_1206_3216Metric_Pad1.30x1.75mm_HandSolder; Link (none) -> https://www.mouser.com/ProductDetail/Vishay-Dale/CRCW120610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; Part Number (none) -> CRCW1206100RFKEA
- R16: footprint (none) -> Resistor_SMD:R_1206_3216Metric_Pad1.30x1.75mm_HandSolder; Link (none) -> https://www.mouser.com/ProductDetail/Vishay-Dale/CRCW120647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; Part Number (none) -> CRCW1206470KFKEA
- U2: footprint Package_CSP:LFCSP-8-1EP_3x3mm_P0.5mm_EP1.45x1.74mm -> Package_SO:SOIC-8_3.9x4.9mm_P1.27mm; Link (none) -> https://www.mouser.com/ProductDetail/Analog-Devices/ADA4622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; Part Number (none) -> ADA4622-2ARZ-R7
Connections:
- net CLAMP_IN: now also D5.2 (A), D6.1 (K), C10.2; no longer D5.1 (K), D6.2 (A)
- net CLAMP_OUT: now also C10.1
- net REF_CLAMP_L: now also U2.5 (+)
- net at D3.1 (K), U2.1: now also D5.1 (K); no longer D6.1 (K)
- net at D4.2 (A), U2.7: now also D6.2 (A); no longer D5.2 (A)
