File: pcb/plugnslay/declick_ref.kicad_sch (KiCad schematic)
At the start: 9 parts, among them U1 ADA4622-2xCP

Commit message: complete first prototype
Parts:
- removed C3: 470n, symbol Device:C
- removed C4: 2.2u, symbol Device:C
- removed R7: 47k, symbol Device:R
- added C8: 2.2u, Capacitor_SMD:C_1206_3216Metric_Pad1.33x1.80mm_HandSolder, symbol Device:C
- added C9: 470n, Capacitor_SMD:C_1206_3216Metric_Pad1.33x1.80mm_HandSolder, symbol Device:C
- added R13: 100k, Resistor_SMD:R_1206_3216Metric_Pad1.30x1.75mm_HandSolder, symbol Device:R
- R10: value 100k -> 47k; footprint (none) -> Resistor_SMD:R_1206_3216Metric_Pad1.30x1.75mm_HandSolder; Link (none) -> https://www.mouser.com/ProductDetail/Vishay-Dale/CRCW120647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; Part Number (none) -> CRCW120647K0FKEA
- R11: value 220k -> 100k; footprint (none) -> Resistor_SMD:R_1206_3216Metric_Pad1.30x1.75mm_HandSolder; Link (none) -> https://www.mouser.com/ProductDetail/Vishay-Dale/CRCW120610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; Part Number (none) -> CRCW1206100KFKEAC
- R12: value 100k -> 220k; footprint (none) -> Resistor_SMD:R_1206_3216Metric_Pad1.30x1.75mm_HandSolder; Link (none) -> https://www.mouser.com/ProductDetail/Vishay-Dale/CRCW120622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; Part Number (none) -> CRCW1206220KFKEA
- R8: value 1k -> 47k; footprint (none) -> Resistor_SMD:R_1206_3216Metric_Pad1.30x1.75mm_HandSolder; Link (none) -> https://www.mouser.com/ProductDetail/Vishay-Dale/CRCW120647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; Part Number (none) -> CRCW120647K0FKEA
- R9: value 47k -> 1k; footprint (none) -> Resistor_SMD:R_1206_3216Metric_Pad1.30x1.75mm_HandSolder; Link (none) -> https://www.mouser.com/ProductDetail/Vishay-Dale/CRCW12061K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; Part Number (none) -> CRCW12061K00FKEA
- U1: footprint Package_CSP:LFCSP-8-1EP_3x3mm_P0.5mm_EP1.45x1.74mm -> Package_SO:SOIC-8_3.9x4.9mm_P1.27mm; Link (none) -> https://www.mouser.com/ProductDetail/Analog-Devices/ADA4622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; Part Number (none) -> ADA4622-2ARZ-R7
Connections:
- net +5V: now also R8.2
- net GND: now also R10.2, R9.1, C8.1, R13.1; no longer R12.1, R8.1, R9.2
- net REF_CLAMP: now also R11.2, C9.1; no longer R10.2
- net REF_CLAMP_H: now also R11.1, R12.2; no longer R10.1, R11.2
- net REF_CLAMP_L: now also R12.1, R13.2; no longer R11.1, R12.2
- net at U1.6 (-): now also R10.1, C9.2; no longer R9.1
- net at U1.5 (+): now also R8.1, R9.2, C8.2; no longer R8.2
