File: pcb/plugnslay/plugnslay.kicad_sch (KiCad schematic)
At the start: 2 parts, among them U1 ADA4622-2xCP, U2 ADA4622-2xCP

Commit message: complete first prototype
Parts:
- added C1, C3: 22n, Capacitor_SMD:C_1206_3216Metric_Pad1.33x1.80mm_HandSolder, symbol Device:C
- added C11: 2.2u, Capacitor_SMD:C_1206_3216Metric_Pad1.33x1.80mm_HandSolder, symbol Device:C
- added C2, C4: 1u, Capacitor_SMD:C_1206_3216Metric_Pad1.33x1.80mm_HandSolder, symbol Device:C
- added J1: AudioJack2_Switch, Connector_Audio:Jack_6.35mm_Neutrik_NRJ4HF_Horizontal, symbol Connector_Audio:AudioJack2_Switch
- added J2: AudioJack3_SwitchTR, Connector_Audio:Jack_3.5mm_CUI_SJ1-3535NG_Horizontal_CircularHoles, symbol Connector_Audio:AudioJack3_SwitchTR
- added J3: USB_C_Receptacle_PowerOnly_6P, Connector_USB:USB_C_Receptacle_GCT_USB4125-xx-x-0190_6P_TopMnt_Horizontal, symbol Connector:USB_C_Receptacle_PowerOnly_6P
- added R17, R18: 4.7k, Resistor_SMD:R_1206_3216Metric_Pad1.30x1.75mm_HandSolder, symbol Device:R
- U1, U2: footprint Package_CSP:LFCSP-8-1EP_3x3mm_P0.5mm_EP1.45x1.74mm -> Package_SO:SOIC-8_3.9x4.9mm_P1.27mm; Link (none) -> https://www.mouser.com/ProductDetail/Analog-Devices/ADA4622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; Part Number (none) -> ADA4622-2ARZ-R7
Connections:
- net +5V: now also C1.1, C11.1, C2.2, C3.1, C4.2, J3.A9 (VBUS), J3.B9 (VBUS)
- net GND: now also C1.2, C11.2, C2.1, C3.2, C4.1, J1.S, J1.SN, J1.TN, J2.RN, J2.S, J2.TN, J3.A12 (GND), J3.B12 (GND), J3.S1 (SHIELD), R17.2, R18.2
- net Input Biasing and Buffer/JACK_IN: now also J1.T
- new net: J3.A5 (CC1), R18.1
- new net: J3.B5 (CC2), R17.1
- new net Output Clamping & Coupling/CLAMP_OUT: J2.R, J2.T
Other:
- sheet Output Clamping & Coupling ports: added CLAMP_IN, CLAMP_OUT; removed none
- moved on the sheet: U2C

Commit message: bom and tweak links
Parts:
- C1, C3: Link https://mou.sr/46W6mYv -> https://www.mouser.com/ProductDetail/KEMET/C1206C223K3RACTU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
Changed lines of the file:
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@@
 			)
 		)
-		(property "Link" "https://mou.sr/46W6mYv"
+		(property "Link" "https://www.mouser.com/ProductDetail/KEMET/C1206C223K3RACTU?qs=nanIO8yDHNwBF9gQ989a6w%3D%3D"
 			(at 207.01 45.72 0)
 			(effects
@@
 			)
 		)
-		(property "Link" "https://mou.sr/46W6mYv"
+		(property "Link" "https://www.mouser.com/ProductDetail/KEMET/C1206C223K3RACTU?qs=nanIO8yDHNwBF9gQ989a6w%3D%3D"
 			(at 156.21 44.45 0)
 			(effects
