File: pcb/plugnslay/input_bias_buffer.kicad_sch (KiCad schematic)
At the start: 14 parts, among them U1 ADA4622-2xCP

Commit message: complete first prototype
Parts:
- removed C1: 1u, symbol Device:C
- removed C2: 2.2n, symbol Device:C
- removed R13: 100, symbol Device:R
- added C6: 3.3n, Capacitor_SMD:C_1206_3216Metric_Pad1.33x1.80mm_HandSolder, symbol Device:C
- added C7: 22n, Capacitor_SMD:C_1206_3216Metric_Pad1.33x1.80mm_HandSolder, symbol Device:C
- added R7: 100, Resistor_SMD:R_1206_3216Metric_Pad1.30x1.75mm_HandSolder, symbol Device:R
- C5: value 22n -> 1u; footprint (none) -> Capacitor_SMD:C_1206_3216Metric_Pad1.33x1.80mm_HandSolder; Link (none) -> https://www.mouser.com/ProductDetail/KEMET/C1206C105K4RAC?q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; Part Number (none) -> C1206C105K4RAC
- D1, D2: footprint (none) -> Diode_SMD:D_SOD-123; Link (none) -> https://www.mouser.com/ProductDetail/Vishay/1N4448W-HE3_A-0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; Part Number (none) -> 1N4448W-HE3_A-08
- R1: footprint (none) -> Resistor_SMD:R_1206_3216Metric_Pad1.30x1.75mm_HandSolder; Link (none) -> https://www.mouser.com/ProductDetail/Vishay-Dale/CRCW120610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; Part Number (none) -> CRCW1206100RFKEA
- R2: footprint (none) -> Resistor_SMD:R_1206_3216Metric_Pad1.30x1.75mm_HandSolder; Link (none) -> https://www.mouser.com/ProductDetail/Vishay-Dale/CRCW12061M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; Part Number (none) -> CRCW12061M00FKEA
- R3, R4: footprint (none) -> Resistor_SMD:R_1206_3216Metric_Pad1.30x1.75mm_HandSolder; Link (none) -> https://www.mouser.com/ProductDetail/Vishay-Dale/CRCW120647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; Part Number (none) -> CRCW1206470KFKEA
- R5: footprint (none) -> Resistor_SMD:R_1206_3216Metric_Pad1.30x1.75mm_HandSolder; Link (none) -> https://www.mouser.com/ProductDetail/Vishay-Dale/CRCW12061K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; Part Number (none) -> CRCW12061K00FKEA
- R6: footprint (none) -> Resistor_SMD:R_1206_3216Metric_Pad1.30x1.75mm_HandSolder; Link (none) -> https://www.mouser.com/ProductDetail/Vishay-Dale/CRCW120610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; Part Number (none) -> CRCW120610K0FKEA
- RV1: footprint Potentiometer_THT:Potentiometer_Alpha_RD901F-40-00D_Single_Vertical_CircularHoles -> Potentiometer_THT:Potentiometer_Bourns_PTV09A-1_Single_Vertical; Link (none) -> https://www.mouser.com/ProductDetail/Bourns/PTV09A-2030F-B5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; Part Number (none) -> PTV09A-2030F-B503
- U1: footprint Package_CSP:LFCSP-8-1EP_3x3mm_P0.5mm_EP1.45x1.74mm -> Package_SO:SOIC-8_3.9x4.9mm_P1.27mm; Link (none) -> https://www.mouser.com/ProductDetail/Analog-Devices/ADA4622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; Part Number (none) -> ADA4622-2ARZ-R7
Connections:
- net GND: now also C6.1, C7.1; no longer C5.1
- net SIG_BUF: now also C7.2, R7.2; no longer C5.2
- net at R3.1, R4.2, R5.1: now also C5.2
- net at U1.1: now also RV1.2, R7.1; no longer RV1.3
- net at R6.2, U1.2 (-): now also RV1.1; no longer RV1.2
- net at D1.2 (A), D2.1 (K), R5.2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: now also C6.2
- net at R1.2, R2.2: now also C5.1

Commit message: bom and tweak links
Parts:
- C7: Link https://mou.sr/46W6mYv -> https://www.mouser.com/ProductDetail/KEMET/C1206C223K3RACTU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
Changed lines of the file:
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@@
 			)
 		)
-		(property "Link" "https://mou.sr/46W6mYv"
+		(property "Link" "https://www.mouser.com/ProductDetail/KEMET/C1206C223K3RACTU?qs=nanIO8yDHNwBF9gQ989a6w%3D%3D"
 			(at 229.87 95.25 0)
 			(effects

Commit message: fix pot ref, gen gerbers
Parts:
- RV1: Link https://www.mouser.com/ProductDetail/Bourns/PTV09A-2030F-B5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 -> https://www.mouser.com/ProductDetail/652-PTV09A2020SB503; Part Number PTV09A-2030F-B503 -> PTV09A-2020S-B503
Changed lines of the file:
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@@
 			)
 		)
-		(property "Part Number" "PTV09A-2030F-B503"
+		(property "Part Number" " PTV09A-2020S-B503"
 			(at 204.47 97.79 0)
 			(effects
@@
 			)
 		)
-		(property "Link" "https://www.mouser.com/ProductDetail/Bourns/PTV09A-2030F-B503?qs=oyIm%2F3giSj7PFvq2byJ%252BHA%3D%3D"
+		(property "Link" "https://www.mouser.com/ProductDetail/652-PTV09A2020SB503"
 			(at 204.47 97.79 0)
 			(effects
