File: pcb/plugnslay/plugnslay.kicad_pcb (KiCad board)
At the start: 2 copper layers, 132.1 x 40.6 mm, 43 parts, among them J1 AudioJack2_Switch, J2 AudioJack3_SwitchTR, J3 USB_C_Receptacle_PowerOnly_6P, U1 ADA4622-2xCP, U2 ADA4622-2xCP

Commit message: fix silk label for power
Other:
- board text added: "← POWER"
- board text removed: "↓ POWER"
Changed lines of the file:
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@@
 		)
 	)
-	(gr_text "↓ POWER"
-		(at 116.078 87.376 0)
+	(gr_text "← POWER"
+		(at 189.484 121.92 0)
 		(layer "F.SilkS")
 		(effects
